File: hardware/ESP32s3APRS.kicad_pcb (KiCad board)
At the start: 2 copper layers, 100 x 62 mm, 156 parts, among them J101 SSQ-108-01-G-S, J102 SSQ-112-01-G-S, J103 SLW-108-01-G-S, J104 SLW-108-01-G-S, J105 HTSW-108-07-G-S, J106 HTSW-108-07-G-S, J107 SLW-108-01-G-S, J108 HTSW-108-07-G-S, J109 HTSW-101-07-G-S, J110 HTSW-101-07-G-S, J111 SLW-101-01-G-S, J112 SLW-101-01-G-S, J201 WR-DC-694108301002, J202 USB4105-GF-A-120, J203 Keystone_1043P, J204 S3B-PH-SM4-TB, J301 U.FL-R-SMT-1, J302 S2B-ZR-SM4A-TF, J501 HTSW-103-07-G-S, J601 FH34SRJ-24S-05SH, J602 U.FL-R-SMT-1, Q101 BC846BW_SOT323, Q102 RZF020P01TL, Q201 BC846BW_SOT323, Q403 RTF025N03TL, Q406 RZF020P01TL, Q501 BC846BW_SOT323, Q603 RTF025N03TL, SW1 SKTDLDE010, SW101 PCM13SMTR, SW2 SKTDLDE010, SW3 SKTDLDE010, U101 AP7361C-33E_SOT223, U102 XC6206P332PR_SOT89, U201 PI3USB102G, U202 MAX77757CEFG+, U301 L86-M33, U401 SA868, U501 ESP32-S3-WROOM-1U, U502 LP2985-3.3

Commit message: hardware : pcb cleanup
Parts:
- JP101, JP102, JP103: value SolderJumper_2_Open -> DNP 0603; footprint Jumper:SolderJumper-2_P1.3mm_Open_RoundedPad1.0x1.5mm -> Resistor_SMD:R_0603_1608Metric_Pad0.98x0.95mm_HandSolder
- moved JP102 0.51 mm to (139.6, 78.3)
- moved JP103 0.51 mm to (123.5, 78.3)
- moved JP101 0.50 mm to (149.0, 78.4)
- moved C402 0.20 mm to (128.2, 78.1)
- moved C401 0.18 mm to (129.9, 78.1)
- moved R402 0.18 mm to (126.5, 78.1)
- moved R401 0.15 mm to (131.5, 78.1)
Routing:
- net GND: track 56.9 -> 60.9 mm, vias 459 -> 462
- net Net-(J108-Pad1): track 85.0 -> 87.7 mm
- net Net-(JP102-Pad2): track 11.3 -> 10.7 mm
- net /USB Charger/Vsys: track 91.6 -> 91.8 mm, vias 21 -> 22
