File: hardware/ESP32s3APRS.kicad_sch (KiCad schematic)
At the start: 52 parts, among them J101 SSQ-108-01-G-S, J102 SSQ-112-01-G-S, J103 SLW-108-01-G-S, J104 SLW-108-01-G-S, J105 HTSW-108-07-G-S, J106 HTSW-108-07-G-S, J107 SLW-108-01-G-S, J108 HTSW-108-07-G-S, J109 HTSW-101-07-G-S, J110 HTSW-101-07-G-S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

Commit message: hardware : pcb cleanup
Parts:
- JP101, JP102, JP103: value SolderJumper_2_Open -> DNP 0603; footprint Jumper:SolderJumper-2_P1.3mm_Open_RoundedPad1.0x1.5mm -> Resistor_SMD:R_0603_1608Metric_Pad0.98x0.95mm_HandSolder
Changed lines of the file:
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@@
     (in_bom yes) (on_board yes)
     (property "Reference" "JP103" (id 0) (at 207.01 129.54 0))
-    (property "Value" "SolderJumper_2_Open" (id 1) (at 184.15 129.54 0))
-    (property "Footprint" "Jumper:SolderJumper-2_P1.3mm_Open_RoundedPad1.0x1.5mm" (id 2) (at 199.39 129.54 0)
+    (property "Value" "DNP 0603" (id 1) (at 184.15 129.54 0))
+    (property "Footprint" "Resistor_SMD:R_0603_1608Metric_Pad0.98x0.95mm_HandSolder" (id 2) (at 199.39 129.54 0)
       (effects (font (size 1.27 1.27)) hide)
     )
@@
     (in_bom yes) (on_board yes)
     (property "Reference" "JP101" (id 0) (at 207.01 113.03 0))
-    (property "Value" "SolderJumper_2_Open" (id 1) (at 184.15 113.03 0))
-    (property "Footprint" "Jumper:SolderJumper-2_P1.3mm_Open_RoundedPad1.0x1.5mm" (id 2) (at 199.39 113.03 0)
+    (property "Value" "DNP 0603" (id 1) (at 184.15 113.03 0))
+    (property "Footprint" "Resistor_SMD:R_0603_1608Metric_Pad0.98x0.95mm_HandSolder" (id 2) (at 199.39 113.03 0)
       (effects (font (size 1.27 1.27)) hide)
     )
@@
     (in_bom yes) (on_board yes)
     (property "Reference" "JP102" (id 0) (at 207.01 121.92 0))
-    (property "Value" "SolderJumper_2_Open" (id 1) (at 184.15 120.65 0))
-    (property "Footprint" "Jumper:SolderJumper-2_P1.3mm_Open_RoundedPad1.0x1.5mm" (id 2) (at 199.39 120.65 0)
+    (property "Value" "DNP 0603" (id 1) (at 184.15 120.65 0))
+    (property "Footprint" "Resistor_SMD:R_0603_1608Metric_Pad0.98x0.95mm_HandSolder" (id 2) (at 199.39 120.65 0)
       (effects (font (size 1.27 1.27)) hide)
     )
@@
     )
     (path "/be8f1ccf-178c-4cda-8589-681ef4a72d48"
-      (reference "JP101") (unit 1) (value "SolderJumper_2_Open") (footprint "Jumper:SolderJumper-2_P1.3mm_Open_RoundedPad1.0x1.5mm")
+      (reference "JP101") (unit 1) (value "DNP 0603") (footprint "Resistor_SMD:R_0603_1608Metric_Pad0.98x0.95mm_HandSolder")
     )
     (path "/f5be40c7-9a88-41e0-89dc-ddf1a501575c"
-      (reference "JP102") (unit 1) (value "SolderJumper_2_Open") (footprint "Jumper:SolderJumper-2_P1.3mm_Open_RoundedPad1.0x1.5mm")
+      (reference "JP102") (unit 1) (value "DNP 0603") (footprint "Resistor_SMD:R_0603_1608Metric_Pad0.98x0.95mm_HandSolder")
     )
     (path "/9b4065f3-acb0-429f-a07b-bf5057d40076"
-      (reference "JP103") (unit 1) (value "SolderJumper_2_Open") (footprint "Jumper:SolderJumper-2_P1.3mm_Open_RoundedPad1.0x1.5mm")
+      (reference "JP103") (unit 1) (value "DNP 0603") (footprint "Resistor_SMD:R_0603_1608Metric_Pad0.98x0.95mm_HandSolder")
     )
     (path "/00000000-0000-0000-0000-0000649ad211/62f35773-c11f-4879-9947-b70cb8e39ac5"
